File: VFD_Clock.kicad_sch (KiCad schematic)
At the start: 42 parts, among them J1 USB_C_Receptacle_USB2.0, Q1 MMBT3904, Q2 MMBT3904, U1 USBLC6-2SC6, U2 CH340C, U3 ESP-M2, U4 MT3608, U5 RT8059GJ5, U6 RT8059GJ5

Commit message: Add new MCU then remove original MCU and 3v3 buck converter
Parts:
- removed C4: 10uF, Capacitor_SMD:C_0805_2012Metric, symbol Device:C_Small
- removed C6: 10pF, Capacitor_SMD:C_0805_2012Metric, symbol Device:C_Small
- removed L3: 4.7uH, Inductor_SMD:L_Taiyo-Yuden_NR-60xx, symbol Device:L_Small
- removed R11: 180k, Resistor_SMD:R_0805_2012Metric, symbol Device:R_Small
- removed R13: 39k, Resistor_SMD:R_0805_2012Metric, symbol Device:R_Small
- removed R14: 1k, Resistor_SMD:R_0805_2012Metric, symbol Device:R_Small
- removed U3: ESP-M2, ESP-M2:ESP-M2, symbol ESP-M2:ESP-M2
- removed U6: RT8059GJ5, Package_TO_SOT_SMD:SOT-23-5, symbol RT8059:RT8059GJ5
- added C1: 10uF, Capacitor_SMD:C_0805_2012Metric, symbol Device:C_Small
- C2: value 100nF -> 10uF
- gave numbers to parts that had none: 1
- renumbered C5 to C4, C1 to C5, C7 to C6, C8 to C7, C9 to C8, C11 to C9, R8 to R10, R15 to R11, R9 to R12, R10 to R6, R12 to R7, R6 to R8, R7 to R9, U2 to U3
Connections:
- net +3V3: now also U2.19 (3V3)
- net +5V: now also U2.11 (5V), U2.8 (5V), C1.2; no longer C10.1
- net DATA: now also U2.3 (G18)
- net GND: now also U2.10 (GND), U2.14 (GND), U2.9 (GND), C1.1
- net GPIO0: now also U2.15 (G0)
- net RST: now also C10.1, U2.16 (EN)
- net RX: now also U2.17 (G3)
- net SH_CP: now also U2.1 (G26)
- net ST_CP: now also U2.4 (G19)
- net TX: now also U2.18 (G1)
- no-connect marks 13 -> 14
Other:
- note added: "Power Caps"
- note removed: "5v to 3.3v Step-Down"
- moved on the sheet: C5, Q1, Q2, R10, R12, R8, R9, U2, U3

Commit message: Clear all ERC errors
Parts:
- RV1: symbol Device:R_POT_Small -> Device:R_Potentiometer_Small
Changed lines of the file:
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@@
   (junction (at 223.52 31.75) (diameter 0) (color 0 0 0 0)
   )
+  (junction (at 270.51 45.72) (diameter 0) (color 0 0 0 0)
+  )
   (junction (at 223.52 26.67) (diameter 0) (color 0 0 0 0)
   )
   (junction (at 257.81 35.56) (diameter 0) (color 0 0 0 0)
   )
+  (junction (at 186.69 137.16) (diameter 0) (color 0 0 0 0)
+  )
+  (junction (at 62.23 118.11) (diameter 0) (color 0 0 0 0)
+  )
   (junction (at 226.06 121.92) (diameter 0) (color 0 0 0 0)
   )
@@
   )
   (junction (at 229.87 44.45) (diameter 0) (color 0 0 0 0)
+  )
+  (junction (at 186.69 142.24) (diameter 0) (color 0 0 0 0)
   )
   (no_connect (at 215.9 133.35))
@@
     (stroke (width 0) (type default) (color 0 0 0 0))
   )
-  (wire (pts (xy 270.51 44.45) (xy 270.51 46.99))
+  (wire (pts (xy 270.51 44.45) (xy 270.51 45.72))
     (stroke (width 0) (type default) (color 0 0 0 0))
   )
@@
   )
   (wire (pts (xy 247.65 44.45) (xy 247.65 26.67))
+    (stroke (width 0) (type default) (color 0 0 0 0))
+  )
+  (wire (pts (xy 270.51 45.72) (xy 270.51 46.99))
     (stroke (width 0) (type default) (color 0 0 0 0))
   )
@@
     (pin "1")
   )
-  (symbol (lib_id "Device:R_POT_Small") (at 257.81 40.64 0) (unit 1)
+  (symbol (lib_id "Device:R_Potentiometer_Small") (at 257.81 40.64 0) (unit 1)
     (in_bom yes) (on_board yes)
     (property "Reference" "RV1" (id 0) (at 256.3114 39.4716 0)
@@
     (pin "2")
   )
+  (symbol (lib_id "power:PWR_FLAG") (at 62.23 118.11 90) (unit 1)
+    (in_bom yes) (on_board yes) (fields_autoplaced)
+    (property "Reference" "#FLG0103" (id 0) (at 60.325 118.11 0)
+      (effects (font (size 1.27 1.27)) hide)
+    )
+    (property "Value" "PWR_FLAG" (id 1) (at 58.42 118.1099 90)
+      (effects (font (size 1.27 1.27)) (justify left) hide)
+    )
+    (property "Footprint" "" (id 2) (at 62.23 118.11 0)
+      (effects (font (size 1.27 1.27)) hide)
+    )
+    (property "Datasheet" "~" (id 3) (at 62.23 118.11 0)
+      (effects (font (size 1.27 1.27)) hide)
+    )
+    (pin "1")
+  )
   (symbol (lib_id "power:+5V") (at 148.59 87.63 90) (unit 1)
     (in_bom yes) (on_board yes)
@@
     (pin "1")
   )
+  (symbol (lib_id "power:PWR_FLAG") (at 186.69 142.24 90) (unit 1)
+    (in_bom yes) (on_board yes) (fields_autoplaced)
+    (property "Reference" "#FLG0102" (id 0) (at 184.785 142.24 0)
+      (effects (font (size 1.27 1.27)) hide)
+    )
+    (property "Value" "PWR_FLAG" (id 1) (at 182.88 142.2399 90)
+      (effects (font (size 1.27 1.27)) (justify left) hide)
+    )
+    (property "Footprint" "" (id 2) (at 186.69 142.24 0)
+      (effects (font (size 1.27 1.27)) hide)
+    )
+    (property "Datasheet" "~" (id 3) (at 186.69 142.24 0)
+      (effects (font (size 1.27 1.27)) hide)
+    )
+    (pin "1")
+  )
   (symbol (lib_id "power:GND") (at 171.45 90.17 90) (unit 1)
     (in_bom yes) (on_board yes)
@@
     )
     (property "Datasheet" "" (id 3) (at 275.59 139.7 0)
+      (effects (font (size 1.27 1.27)) hide)
+    )
+    (pin "1")
+  )
+  (symbol (lib_id "power:PWR_FLAG") (at 186.69 137.16 90) (unit 1)
+    (in_bom yes) (on_board yes) (fields_autoplaced)
+    (property "Reference" "#FLG0101" (id 0) (at 184.785 137.16 0)
+      (effects (font (size 1.27 1.27)) hide)
+    )
+    (property "Value" "PWR_FLAG" (id 1) (at 182.88 137.1599 90)
+      (effects (font (size 1.27 1.27)) (justify left) hide)
+    )
+    (property "Footprint" "" (id 2) (at 186.69 137.16 0)
+      (effects (font (size 1.27 1.27)) hide)
+    )
+    (property "Datasheet" "~" (id 3) (at 186.69 137.16 0)
       (effects (font (size 1.27 1.27)) hide)
     )
@@
     (pin "1")
   )
+  (symbol (lib_id "power:PWR_FLAG") (at 270.51 45.72 270) (unit 1)
+    (in_bom yes) (on_board yes) (fields_autoplaced)
+    (property "Reference" "#FLG01" (id 0) (at 272.415 45.72 0)
+      (effects (font (size 1.27 1.27)) hide)
+    )
+    (property "Value" "PWR_FLAG" (id 1) (at 274.32 45.7201 90)
+      (effects (font (size 1.27 1.27)) (justify left) hide)
+    )
+    (property "Footprint" "" (id 2) (at 270.51 45.72 0)
+      (effects (font (size 1.27 1.27)) hide)
+    )
+    (property "Datasheet" "~" (id 3) (at 270.51 45.72 0)
+      (effects (font (size 1.27 1.27)) hide)
+    )
+    (pin "1")
+  )
   (symbol (lib_id "Device:C_Small") (at 194.31 139.7 180) (unit 1)
     (in_bom yes) (on_board yes)
@@
   )
   (symbol_instances
+    (path "/dda5ca94-84bd-44f1-835a-53b729636e5b"
+      (reference "#FLG01") (unit 1) (value "PWR_FLAG") (footprint "")
+    )
+    (path "/59fd5e49-0184-462c-9c09-bce6e7d9d843"
+      (reference "#FLG0101") (unit 1) (value "PWR_FLAG") (footprint "")
+    )
+    (path "/2b35b0b7-ee1d-4bf5-8946-6bbdb265ea32"
+      (reference "#FLG0102") (unit 1) (value "PWR_FLAG") (footprint "")
+    )
+    (path "/1b5212fa-743a-47ed-a304-7d164657f2d6"
+      (reference "#FLG0103") (unit 1) (value "PWR_FLAG") (footprint "")
+    )
     (path "/00000000-0000-0000-0000-000060ae325d"
       (reference "#PWR01") (unit 1) (value "GND") (footprint "")

Commit message: Add in footprint for pot. and start adding some LCSC part numbers
Parts:
- F1: LCSC Part # (none) -> C80270
- J1: LCSC Part # (none) -> C165948
- RV1: footprint Resistor_SMD:R_0805_2012Metric -> BOURNS-3362P:BOURNS-3362P; LCSC Part # (none) -> C111655
- U1: LCSC Part # (none) -> C2827654
- U2: footprint (none) -> StampPico:StampPico; LCSC Part # (none) -> -
- U3: LCSC Part # (none) -> C84681
Changed lines of the file:
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@@
+      (effects (font (size 1.27 1.27)) hide)
+    )
+    (property "LCSC Part #" "C165948" (id 4) (at 39.37 135.89 0)
       (effects (font (size 1.27 1.27)) hide)
     )
@@
       (effects (font (size 1.27 1.27)) hide)
     )
+    (property "LCSC Part #" "C80270" (id 4) (at 71.12 120.65 0)
+      (effects (font (size 1.27 1.27)) hide)
+    )
     (pin "1")
     (pin "2")
@@
     )
     (property "Datasheet" "https://www.st.com/resource/en/datasheet/usblc6-2.pdf" (id 3) (at 90.17 142.24 0)
+      (effects (font (size 1.27 1.27)) hide)
+    )
+    (property "LCSC Part #" "C2827654" (id 4) (at 81.28 137.16 0)
       (effects (font (size 1.27 1.27)) hide)
     )
@@
       (effects (font (size 1.27 1.27)) (justify right))
     )
-    (property "Footprint" "Resistor_SMD:R_0805_2012Metric" (id 2) (at 257.81 40.64 0)
-      (effects (font (size 1.27 1.27)) hide)
-    )
-    (property "Datasheet" "~" (id 3) (at 257.81 40.64 0)
+    (property "Footprint" "BOURNS-3362P:BOURNS-3362P" (id 2) (at 257.81 40.64 0)
+      (effects (font (size 1.27 1.27)) hide)
+    )
+    (property "Datasheet" "https://datasheet.lcsc.com/lcsc/1810162216_BOURNS-3362P-1-204LF_C111655.pdf" (id 3) (at 257.81 40.64 0)
+      (effects (font (size 1.27 1.27)) hide)
+    )
+    (property "LCSC Part #" "C111655" (id 4) (at 257.81 40.64 0)
       (effects (font (size 1.27 1.27)) hide)
     )
@@
     )
     (property "Datasheet" "https://datasheet.lcsc.com/szlcsc/Jiangsu-Qin-Heng-CH340C_C84681.pdf" (id 3) (at 217.17 120.65 0)
+      (effects (font (size 1.27 1.27)) hide)
+    )
+    (property "LCSC Part #" "C84681" (id 4) (at 226.06 140.97 0)
       (effects (font (size 1.27 1.27)) hide)
     )
@@
     (property "Reference" "U2" (id 0) (at 159.385 63.5 0))
     (property "Value" "StampPico" (id 1) (at 159.385 66.04 0))
-    (property "Footprint" "" (id 2) (at 148.59 72.39 0)
+    (property "Footprint" "StampPico:StampPico" (id 2) (at 148.59 72.39 0)
       (effects (font (size 1.27 1.27)) hide)
     )
     (property "Datasheet" "" (id 3) (at 148.59 72.39 0)
+      (effects (font (size 1.27 1.27)) hide)
+    )
+    (property "LCSC Part #" "-" (id 4) (at 160.02 81.28 0)
       (effects (font (size 1.27 1.27)) hide)
     )
@@
     )
     (path "/00000000-0000-0000-0000-000060bbcec9"
-      (reference "RV1") (unit 1) (value "200k") (footprint "Resistor_SMD:R_0805_2012Metric")
+      (reference "RV1") (unit 1) (value "200k") (footprint "BOURNS-3362P:BOURNS-3362P")
     )
     (path "/00000000-0000-0000-0000-000060af3c49"
@@
     )
     (path "/8c68ccd3-e007-4da8-818b-511230f39897"
-      (reference "U2") (unit 1) (value "StampPico") (footprint "")
+      (reference "U2") (unit 1) (value "StampPico") (footprint "StampPico:StampPico")
     )
     (path "/00000000-0000-0000-0000-000060cc759f"

Commit message: Added some more LCSC part numbers
Parts:
- C1, C10, C2, C3, C7, C8, C9: Ext Part (none) -> N; LCSC Part # (none) -> C440198
- C4, C6: Ext Part (none) -> N; LCSC Part # (none) -> C1785
- C5: Ext Part (none) -> N; LCSC Part # (none) -> C49678
- D1: footprint Diode_SMD:D_SMA_Handsoldering -> Diode_SMD:D_SOD-323_HandSoldering; Ext Part (none) -> N; LCSC Part # (none) -> C191023
- F1, J1, U3: Ext Part (none) -> Y
- L1: Ext Part (none) -> OOS; LCSC Part # (none) -> C520365
- L2: footprint Inductor_SMD:L_Taiyo-Yuden_NR-60xx -> Potentiometer_SMD:Potentiometer_ACP_CA6-VSMD_Vertical; Ext Part (none) -> Y; LCSC Part # (none) -> C520369
- Q1, Q2: LCSC Part # (none) -> C20526
- RV1: footprint BOURNS-3362P:BOURNS-3362P -> (none); Ext Part (none) -> Y; LCSC Part # C111655 -> C128551
Changed lines of the file:
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@@
       (effects (font (size 1.27 1.27)) hide)
     )
-    (property "Datasheet" "https://www.usb.org/sites/default/files/documents/usb_type-c.zip" (id 3) (at 43.18 135.89 0)
+    (property "Datasheet" "https://datasheet.lcsc.com/lcsc/2108131730_Korean-Hroparts-Elec-TYPE-C-31-M-12_C165948.pdf" (id 3) (at 43.18 135.89 0)
       (effects (font (size 1.27 1.27)) hide)
     )
     (property "LCSC Part #" "C165948" (id 4) (at 39.37 135.89 0)
+      (effects (font (size 1.27 1.27)) hide)
+    )
+    (property "Ext Part" "Y" (id 5) (at 39.37 135.89 0)
       (effects (font (size 1.27 1.27)) hide)
     )
@@
       (effects (font (size 1.27 1.27)) hide)
     )
-    (property "Datasheet" "~" (id 3) (at 71.12 120.65 0)
+    (property "Datasheet" "https://datasheet.lcsc.com/lcsc/1809191943_Littelfuse-0805L100WR_C80270.pdf" (id 3) (at 71.12 120.65 0)
       (effects (font (size 1.27 1.27)) hide)
     )
     (property "LCSC Part #" "C80270" (id 4) (at 71.12 120.65 0)
+      (effects (font (size 1.27 1.27)) hide)
+    )
+    (property "Ext Part" "Y" (id 5) (at 71.12 120.65 0)
       (effects (font (size 1.27 1.27)) hide)
     )
@@
       (effects (font (size 1.27 1.27)) hide)
     )
+    (property "Ext Part" "N" (id 4) (at 270.51 96.52 0)
+      (effects (font (size 1.27 1.27)) hide)
+    )
+    (property "LCSC Part #" "C440198" (id 5) (at 270.51 96.52 0)
+      (effects (font (size 1.27 1.27)) hide)
+    )
     (pin "1")
     (pin "2")
@@
     (property "Reference" "L2" (id 0) (at 240.03 91.9226 90))
     (property "Value" "4.7uH" (id 1) (at 240.03 94.234 90))
-    (property "Footprint" "Inductor_SMD:L_Taiyo-Yuden_NR-60xx" (id 2) (at 240.03 96.52 0)
+    (property "Footprint" "Potentiometer_SMD:Potentiometer_ACP_CA6-VSMD_Vertical" (id 2) (at 240.03 96.52 0)
       (effects (font (size 1.27 1.27)) hide)
     )
@@
       (effects (font (size 1.27 1.27)) hide)
     )
+    (property "Ext Part" "Y" (id 4) (at 240.03 96.52 0)
+      (effects (font (size 1.27 1.27)) hide)
+    )
+    (property "LCSC Part #" "C520369" (id 5) (at 240.03 96.52 0)
+      (effects (font (size 1.27 1.27)) hide)
+    )
     (pin "1")
     (pin "2")
@@
     )
     (property "Datasheet" "~" (id 3) (at 226.06 87.63 0)
+      (effects (font (size 1.27 1.27)) hide)
+    )
+    (property "Ext Part" "N" (id 4) (at 226.06 87.63 0)
+      (effects (font (size 1.27 1.27)) hide)
+    )
+    (property "LCSC Part #" "C1785" (id 5) (at 226.06 87.63 0)
       (effects (font (size 1.27 1.27)) hide)
     )
@@
     )
     (property "Datasheet" "~" (id 3) (at 220.98 99.06 0)
+      (effects (font (size 1.27 1.27)) hide)
+    )
+    (property "Ext Part" "N" (id 4) (at 220.98 99.06 0)
+      (effects (font (size 1.27 1.27)) hide)
+    )
+    (property "LCSC Part #" "C440198" (id 5) (at 220.98 99.06 0)
       (effects (font (size 1.27 1.27)) hide)
     )
@@
       (effects (font (size 1.27 1.27)) hide)
     )
+    (property "Ext Part" "N" (id 4) (at 229.87 41.91 0)
+      (effects (font (size 1.27 1.27)) hide)
+    )
+    (property "LCSC Part #" "C1785" (id 5) (at 229.87 41.91 0)
+      (effects (font (size 1.27 1.27)) hide)
+    )
     (pin "1")
     (pin "2")
@@
       (effects (font (size 1.27 1.27)) hide)
     )
+    (property "Ext Part" "OOS" (id 4) (at 237.49 44.45 0)
+      (effects (font (size 1.27 1.27)) hide)
+    )
+    (property "LCSC Part #" "C520365" (id 5) (at 237.49 44.45 0)
+      (effects (font (size 1.27 1.27)) hide)
+    )
     (pin "1")
     (pin "2")
@@
     (property "Reference" "D1" (id 0) (at 254 49.7078 0))
     (property "Value" "D_Schottky_Small" (id 1) (at 254 47.3964 0))
-    (property "Footprint" "Diode_SMD:D_SMA_Handsoldering" (id 2) (at 254 44.45 90)
-      (effects (font (size 1.27 1.27)) hide)
-    )
-    (property "Datasheet" "~" (id 3) (at 254 44.45 90)
+    (property "Footprint" "Diode_SMD:D_SOD-323_HandSoldering" (id 2) (at 254 44.45 90)
+      (effects (font (size 1.27 1.27)) hide)
+    )
+    (property "Datasheet" "https://datasheet.lcsc.com/lcsc/1810202112_Guangdong-Hottech-1N5819WS_C191023.pdf" (id 3) (at 254 44.45 90)
+      (effects (font (size 1.27 1.27)) hide)
+    )
+    (property "LCSC Part #" "C191023" (id 4) (at 254 44.45 0)
+      (effects (font (size 1.27 1.27)) hide)
+    )
+    (property "Ext Part" "N" (id 5) (at 254 44.45 0)
       (effects (font (size 1.27 1.27)) hide)
     )
@@
       (effects (font (size 1.27 1.27)) (justify right))
     )
-    (property "Footprint" "BOURNS-3362P:BOURNS-3362P" (id 2) (at 257.81 40.64 0)
-      (effects (font (size 1.27 1.27)) hide)
-    )
-    (property "Datasheet" "https://datasheet.lcsc.com/lcsc/1810162216_BOURNS-3362P-1-204LF_C111655.pdf" (id 3) (at 257.81 40.64 0)
-      (effects (font (size 1.27 1.27)) hide)
-    )
-    (property "LCSC Part #" "C111655" (id 4) (at 257.81 40.64 0)
+    (property "Footprint" "" (id 2) (at 257.81 40.64 0)
+      (effects (font (size 1.27 1.27)) hide)
+    )
+    (property "Datasheet" "https://datasheet.lcsc.com/lcsc/1810170727_HDK-Hokuriku-Elec-Industry-VG039NCHXTB204_C128551.pdf" (id 3) (at 257.81 40.64 0)
+      (effects (font (size 1.27 1.27)) hide)
+    )
+    (property "LCSC Part #" "C128551" (id 4) (at 257.81 40.64 0)
+      (effects (font (size 1.27 1.27)) hide)
+    )
+    (property "Ext Part" "Y" (id 5) (at 257.81 40.64 0)
       (effects (font (size 1.27 1.27)) hide)
     )
@@
       (effects (font (size 1.27 1.27)) hide)
     )
+    (property "Ext Part" "N" (id 4) (at 264.16 40.64 0)
+      (effects (font (size 1.27 1.27)) hide)
+    )
+    (property "LCSC Part #" "C440198" (id 5) (at 264.16 40.64 0)
+      (effects (font (size 1.27 1.27)) hide)
+    )
     (pin "1")
     (pin "2")
@@
     )
     (property "Datasheet" "~" (id 3) (at 271.78 40.64 0)
+      (effects (font (size 1.27 1.27)) hide)
+    )
+    (property "Ext Part" "N" (id 4) (at 271.78 40.64 0)
+      (effects (font (size 1.27 1.27)) hide)
+    )
+    (property "LCSC Part #" "C440198" (id 5) (at 271.78 40.64 0)
       (effects (font (size 1.27 1.27)) hide)
     )
@@
     )
     (property "LCSC Part #" "C84681" (id 4) (at 226.06 140.97 0)
+      (effects (font (size 1.27 1.27)) hide)
+    )
+    (property "Ext Part" "Y" (id 5) (at 226.06 140.97 0)
       (effects (font (size 1.27 1.27)) hide)
     )
@@
       (effects (font (size 1.27 1.27)) hide)
     )
+    (property "Ext Part" "N" (id 4) (at 228.6 121.92 0)
+      (effects (font (size 1.27 1.27)) hide)
+    )
+    (property "LCSC Part #" "C49678" (id 5) (at 228.6 121.92 0)
+      (effects (font (size 1.27 1.27)) hide)
+    )
     (pin "1")
     (pin "2")
@@
       (effects (font (size 1.27 1.27) italic) (justify left) hide)
     )
-    (property "Datasheet" "https://www.fairchildsemi.com/datasheets/2N/2N3904.pdf" (id 3) (at 269.24 147.32 0)
+    (property "Datasheet" "https://datasheet.lcsc.com/lcsc/1811011934_Changjiang-Electronics-Tech--CJ-MMBT3904_C20526.pdf" (id 3) (at 269.24 147.32 0)
       (effects (font (size 1.27 1.27)) (justify left) hide)
+    )
+    (property "LCSC Part #" "C20526" (id 4) (at 269.24 147.32 0)
+      (effects (font (size 1.27 1.27)) hide)
     )
     (pin "1")
@@
       (effects (font (size 1.27 1.27) italic) (justify left) hide)
     )
-    (property "Datasheet" "https://www.fairchildsemi.com/datasheets/2N/2N3904.pdf" (id 3) (at 254 147.32 0)
+    (property "Datasheet" "https://datasheet.lcsc.com/lcsc/1811011934_Changjiang-Electronics-Tech--CJ-MMBT3904_C20526.pdf" (id 3) (at 254 147.32 0)
       (effects (font (size 1.27 1.27)) (justify left) hide)
     )
+    (property "LCSC Part #" "C20526" (id 4) (at 254 147.32 0)
+      (effects (font (size 1.27 1.27)) hide)
+    )
     (pin "1")
     (pin "2")
@@
     )
     (property "Datasheet" "~" (id 3) (at 186.69 139.7 0)
+      (effects (font (size 1.27 1.27)) hide)
+    )
+    (property "Ext Part" "N" (id 4) (at 186.69 139.7 0)
+      (effects (font (size 1.27 1.27)) hide)
+    )
+    (property "LCSC Part #" "C440198" (id 5) (at 186.69 139.7 0)
       (effects (font (size 1.27 1.27)) hide)
     )
@@
       (effects (font (size 1.27 1.27)) hide)
     )
+    (property "Ext Part" "N" (id 4) (at 275.59 143.51 0)
+      (effects (font (size 1.27 1.27)) hide)
+    )
+    (property "LCSC Part #" "C440198" (id 5) (at 275.59 143.51 0)
+      (effects (font (size 1.27 1.27)) hide)
+    )
     (pin "1")
     (pin "2")
@@
     )
     (property "Datasheet" "~" (id 3) (at 194.31 139.7 0)
+      (effects (font (size 1.27 1.27)) hide)
+    )
+    (property "Ext Part" "N" (id 4) (at 194.31 139.7 0)
+      (effects (font (size 1.27 1.27)) hide)
+    )
+    (property "LCSC Part #" "C440198" (id 5) (at 194.31 139.7 0)
       (effects (font (size 1.27 1.27)) hide)
     )
@@
     )
     (path "/00000000-0000-0000-0000-000060ba8172"
-      (reference "D1") (unit 1) (value "D_Schottky_Small") (footprint "Diode_SMD:D_SMA_Handsoldering")
+      (reference "D1") (unit 1) (value "D_Schottky_Small") (footprint "Diode_SMD:D_SOD-323_HandSoldering")
     )
     (path "/00000000-0000-0000-0000-000060ae916f"
@@
     )
     (path "/00000000-0000-0000-0000-000060b681c8"
-      (reference "L2") (unit 1) (value "4.7uH") (footprint "Inductor_SMD:L_Taiyo-Yuden_NR-60xx")
+      (reference "L2") (unit 1) (value "4.7uH") (footprint "Potentiometer_SMD:Potentiometer_ACP_CA6-VSMD_Vertical")
     )
     (path "/00000000-0000-0000-0000-000060d4a6b1"
@@
     )
     (path "/00000000-0000-0000-0000-000060bbcec9"
-      (reference "RV1") (unit 1) (value "200k") (footprint "BOURNS-3362P:BOURNS-3362P")
+      (reference "RV1") (unit 1) (value "200k") (footprint "")
     )
     (path "/00000000-0000-0000-0000-000060af3c49"

Commit message: Add 100k pulldown for filament traces and add more LCSC part numbers
Parts:
- R1, R2: Ext Part (none) -> N; LCSC Part # (none) -> C27834
- R10, R12: Ext Part (none) -> N; LCSC Part # (none) -> C17414
- R11: Ext Part (none) -> N; LCSC Part # (none) -> C26010
- R3: Ext Part (none) -> N; LCSC Part # (none) -> C4310
- R4, R5: Ext Part (none) -> N; LCSC Part # (none) -> C17544
- R6: Ext Part (none) -> N; LCSC Part # (none) -> C149504
- R7: Ext Part (none) -> N; LCSC Part # (none) -> C17501
- R8, R9: Ext Part (none) -> N; LCSC Part # (none) -> C17513
